File: eagle/teensy/teensy.sch (EAGLE design)
At the start: 8 parts

Commit message: new file:   eagle/sensors/sensors.brd
Parts:
- removed J2, J6, REG: (no value), SparkFun-Connectors:CONN_031X03_NO_SILK
- removed J3, J4: (no value), SparkFun-Connectors:CONN_05NO_SILK
- added U$3: 1X8, headers(2mm):1X8
- J1: device SparkFun-Connectors:CONN_031X03_NO_SILK -> SparkFun-Connectors:CONN_041X04_NO_SILK
- U$2: value TINYPICO-NANO-CONNECTOR -> 1X3; device TinyPICO_NANO_Eagle:TINYPICO-NANO-CONNECTOR -> headers(2mm):1X3
Connections:
- removed net INT: J1.1
- new net CS: U$3.8
- new net MISO: U$3.5
- new net MOSI: U$3.6
- new net SBUS: U$2.3
- new net SCK: U$3.7
- net 3V3: now also U$3.1; no longer J3.4, J6.3
- net 5V: now also J1.4, U$2.2; no longer J6.1, REG.3
- net GND: now also J1.3, U$2.1, U$3.2; no longer J3.5, J6.2, REG.2
- net SCL: now also U$3.3; no longer J1.2, J3.2
- net SDA: now also U$3.4; no longer J1.3, J3.1
- net VBAT: now also J1.2; no longer REG.1
Changed lines of the file:
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@@
 <parts>
 <part name="U$1" library="TEENSY 4.0" deviceset="TEENSY_4.0" device=""/>
-<part name="J1" library="SparkFun-Connectors" deviceset="CONN_03" device="1X03_NO_SILK"/>
-<part name="J2" library="SparkFun-Connectors" deviceset="CONN_03" device="1X03_NO_SILK"/>
-<part name="J3" library="SparkFun-Connectors" deviceset="CONN_05" device="NO_SILK"/>
-<part name="J4" library="SparkFun-Connectors" deviceset="CONN_05" device="NO_SILK"/>
-<part name="J6" library="SparkFun-Connectors" deviceset="CONN_03" device="1X03_NO_SILK"/>
-<part name="REG" library="SparkFun-Connectors" deviceset="CONN_03" device="1X03_NO_SILK"/>
-<part name="U$2" library="TinyPICO_NANO_Eagle" deviceset="TINYPICO-NANO-CONNECTOR" device=""/>
+<part name="J1" library="SparkFun-Connectors" deviceset="CONN_04" device="1X04_NO_SILK"/>
+<part name="U$2" library="headers(2mm)" deviceset="1X3" device=""/>
+<part name="U$3" library="headers(2mm)" deviceset="1X8" device=""/>
 </parts>
 <sheets>
@@
 <instances>
 <instance part="U$1" gate="G$1" x="86.36" y="63.5" smashed="yes"/>
-<instance part="J1" gate="J1" x="-10.16" y="93.98" smashed="yes">
-<attribute name="VALUE" x="-12.7" y="86.614" size="1.778" layer="96" font="vector"/>
-<attribute name="NAME" x="-12.7" y="99.568" size="1.778" layer="95" font="vector"/>
+<instance part="J1" gate="J1" x="30.48" y="35.56" smashed="yes">
+<attribute name="VALUE" x="25.4" y="28.194" size="1.778" layer="96" font="vector"/>
+<attribute name="NAME" x="25.4" y="43.688" size="1.778" layer="95" font="vector"/>
 </instance>
-<instance part="J2" gate="J1" x="-10.16" y="73.66" smashed="yes">
-<attribute name="VALUE" x="-12.7" y="66.294" size="1.778" layer="96" font="vector"/>
-<attribute name="NAME" x="-12.7" y="79.248" size="1.778" layer="95" font="vector"/>
+<instance part="U$2" gate="G$1" x="30.48" y="17.78" smashed="yes">
+<attribute name="NAME" x="27.94" y="23.495" size="1.27" layer="95" font="vector"/>
+<attribute name="VALUE" x="27.94" y="10.795" size="1.27" layer="96" font="vector"/>
 </instance>
-<instance part="J3" gate="J1" x="-10.16" y="43.18" smashed="yes">
-<attribute name="VALUE" x="-12.7" y="33.274" size="1.778" layer="96" font="vector"/>
-<attribute name="NAME" x="-12.7" y="51.308" size="1.778" layer="95" font="vector"/>
+<instance part="U$3" gate="G$1" x="27.94" y="66.04" smashed="yes">
+<attribute name="NAME" x="25.4" y="79.375" size="1.27" layer="95" font="vector"/>
+<attribute name="VALUE" x="25.4" y="53.975" size="1.27" layer="96" font="vector"/>
 </instance>
-<instance part="J4" gate="J1" x="-10.16" y="12.7" smashed="yes">
-<attribute name="VALUE" x="-12.7" y="2.794" size="1.778" layer="96" font="vector"/>
-<attribute name="NAME" x="-12.7" y="20.828" size="1.778" layer="95" font="vector"/>
-</instance>
-<instance part="J6" gate="J1" x="7.62" y="73.66" smashed="yes">
-<attribute name="VALUE" x="5.08" y="66.294" size="1.778" layer="96" font="vector"/>
-<attribute name="NAME" x="5.08" y="79.248" size="1.778" layer="95" font="vector"/>
-</instance>
-<instance part="REG" gate="J1" x="27.94" y="53.34" smashed="yes">
-<attribute name="VALUE" x="25.4" y="45.974" size="1.778" layer="96" font="vector"/>
-<attribute name="NAME" x="25.4" y="58.928" size="1.778" layer="95" font="vector"/>
-</instance>
-<instance part="U$2" gate="G$1" x="83.82" y="134.62" smashed="yes"/>
 </instances>
 <busses>
 </busses>
 <nets>
+<net name="GND" class="0">
+<segment>
+<pinref part="J1" gate="J1" pin="3"/>
+<wire x1="35.56" y1="38.1" x2="40.64" y2="38.1" width="0.1524" layer="91"/>
+<label x="35.56" y="38.1" size="1.778" layer="95"/>
+</segment>
+<segment>
+<pinref part="U$2" gate="G$1" pin="1"/>
+<wire x1="33.02" y1="20.32" x2="38.1" y2="20.32" width="0.1524" layer="91"/>
+<label x="35.56" y="20.32" size="1.778" layer="95"/>
+</segment>
+<segment>
+<pinref part="U$3" gate="G$1" pin="2"/>
+<wire x1="30.48" y1="73.66" x2="35.56" y2="73.66" width="0.1524" layer="91"/>
+<label x="33.02" y="73.66" size="1.778" layer="95"/>
+</segment>
+</net>
+<net name="5V" class="0">
+<segment>
+<pinref part="J1" gate="J1" pin="4"/>
+<wire x1="35.56" y1="40.64" x2="40.64" y2="40.64" width="0.1524" layer="91"/>
+<label x="35.56" y="40.64" size="1.778" layer="95"/>
+</segment>
+<segment>
+<pinref part="U$2" gate="G$1" pin="2"/>
+<wire x1="33.02" y1="17.78" x2="38.1" y2="17.78" width="0.1524" layer="91"/>
+<label x="35.56" y="17.78" size="1.778" layer="95"/>
+</segment>
+</net>
+<net name="VBAT" class="0">
+<segment>
+<pinref part="J1" gate="J1" pin="2"/>
+<wire x1="35.56" y1="35.56" x2="40.64" y2="35.56" width="0.1524" layer="91"/>
+<label x="35.56" y="35.56" size="1.778" layer="95"/>
+</segment>
+</net>
+<net name="SBUS" class="0">
+<segment>
+<pinref part="U$2" gate="G$1" pin="3"/>
+<wire x1="33.02" y1="15.24" x2="38.1" y2="15.24" width="0.1524" layer="91"/>
+<label x="35.56" y="15.24" size="1.778" layer="95"/>
+</segment>
+</net>
 <net name="3V3" class="0">
 <segment>
-<pinref part="J3" gate="J1" pin="4"/>
-<wire x1="-2.54" y1="45.72" x2="5.08" y2="45.72" width="0.1524" layer="91"/>
-<label x="-2.54" y="45.72" size="1.778" layer="95"/>
-</segment>
-<segment>
-<pinref part="J6" gate="J1" pin="3"/>
-<wire x1="15.24" y1="76.2" x2="20.32" y2="76.2" width="0.1524" layer="91"/>
-<label x="15.24" y="76.2" size="1.778" layer="95"/>
+<pinref part="U$3" gate="G$1" pin="1"/>
+<wire x1="30.48" y1="76.2" x2="35.56" y2="76.2" width="0.1524" layer="91"/>
+<label x="33.02" y="76.2" size="1.778" layer="95"/>
 </segment>
 </net>
-<net name="GND" class="0">
+<net name="SCL" class="0">
 <segment>
-<pinref part="J3" gate="J1" pin="5"/>
-<wire x1="-2.54" y1="48.26" x2="5.08" y2="48.26" width="0.1524" layer="91"/>
-<label x="-2.54" y="48.26" size="1.778" layer="95"/>
-</segment>
-<segment>
-<pinref part="J6" gate="J1" pin="2"/>
-<wire x1="15.24" y1="73.66" x2="20.32" y2="73.66" width="0.1524" layer="91"/>
-<label x="15.24" y="73.66" size="1.778" layer="95"/>
-</segment>
-<segment>
-<pinref part="REG" gate="J1" pin="2"/>
-<wire x1="35.56" y1="53.34" x2="40.64" y2="53.34" width="0.1524" layer="91"/>
-<label x="35.56" y="53.34" size="1.778" layer="95"/>
+<pinref part="U$3" gate="G$1" pin="3"/>
+<wire x1="30.48" y1="71.12" x2="35.56" y2="71.12" width="0.1524" layer="91"/>
+<label x="33.02" y="71.12" size="1.778" layer="95"/>
 </segment>
 </net>
 <net name="SDA" class="0">
 <segment>
-<pinref part="J1" gate="J1" pin="3"/>
-<wire x1="-2.54" y1="96.52" x2="2.54" y2="96.52" width="0.1524" layer="91"/>
-<label x="-2.54" y="96.52" size="1.778" layer="95"/>
-</segment>
-<segment>
-<pinref part="J3" gate="J1" pin="1"/>
-<wire x1="-2.54" y1="38.1" x2="5.08" y2="38.1" width="0.1524" layer="91"/>
-<label x="-2.54" y="38.1" size="1.778" layer="95"/>
+<pinref part="U$3" gate="G$1" pin="4"/>
+<wire x1="30.48" y1="68.58" x2="35.56" y2="68.58" width="0.1524" layer="91"/>
+<label x="33.02" y="68.58" size="1.778" layer="95"/>
 </segment>
 </net>
-<net name="SCL" class="0">
+<net name="MISO" class="0">
 <segment>
-<pinref part="J1" gate="J1" pin="2"/>
-<wire x1="-2.54" y1="93.98" x2="2.54" y2="93.98" width="0.1524" layer="91"/>
-<label x="-2.54" y="93.98" size="1.778" layer="95"/>
-</segment>
-<segment>
-<pinref part="J3" gate="J1" pin="2"/>
-<wire x1="-2.54" y1="40.64" x2="5.08" y2="40.64" width="0.1524" layer="91"/>
-<label x="-2.54" y="40.64" size="1.778" layer="95"/>
+<pinref part="U$3" gate="G$1" pin="5"/>
+<wire x1="30.48" y1="66.04" x2="35.56" y2="66.04" width="0.1524" layer="91"/>
+<label x="33.02" y="66.04" size="1.778" layer="95"/>
 </segment>
 </net>
-<net name="INT" class="0">
+<net name="MOSI" class="0">
 <segment>
-<pinref part="J1" gate="J1" pin="1"/>
-<wire x1="-2.54" y1="91.44" x2="2.54" y2="91.44" width="0.1524" layer="91"/>
-<label x="-2.54" y="91.44" size="1.778" layer="95"/>
+<pinref part="U$3" gate="G$1" pin="6"/>
+<wire x1="30.48" y1="63.5" x2="35.56" y2="63.5" width="0.1524" layer="91"/>
+<label x="33.02" y="63.5" size="1.778" layer="95"/>
 </segment>
 </net>
-<net name="5V" class="0">
+<net name="SCK" class="0">
 <segment>
-<pinref part="J6" gate="J1" pin="1"/>
-<wire x1="15.24" y1="71.12" x2="20.32" y2="71.12" width="0.1524" layer="91"/>
-<label x="15.24" y="71.12" size="1.778" layer="95"/>
-</segment>
-<segment>
-<pinref part="REG" gate="J1" pin="3"/>
-<wire x1="35.56" y1="55.88" x2="40.64" y2="55.88" width="0.1524" layer="91"/>
-<label x="35.56" y="55.88" size="1.778" layer="95"/>
+<pinref part="U$3" gate="G$1" pin="7"/>
+<wire x1="30.48" y1="60.96" x2="35.56" y2="60.96" width="0.1524" layer="91"/>
+<label x="33.02" y="60.96" size="1.778" layer="95"/>
 </segment>
 </net>
-<net name="VBAT" class="0">
+<net name="CS" class="0">
 <segment>
-<pinref part="REG" gate="J1" pin="1"/>
-<wire x1="35.56" y1="50.8" x2="40.64" y2="50.8" width="0.1524" layer="91"/>
-<label x="35.56" y="50.8" size="1.778" layer="95"/>
+<pinref part="U$3" gate="G$1" pin="8"/>
+<wire x1="30.48" y1="58.42" x2="35.56" y2="58.42" width="0.1524" layer="91"/>
+<label x="33.02" y="58.42" size="1.778" layer="95"/>
 </segment>
 </net>
