File: eagle/sensors/sensors.sch (EAGLE design)
At the start: 8 parts

Commit message: modified:   eagle/sensors/sensors.brd
Connections:
- net CS: now also U$1.5; no longer U$1.8
- net MISO: now also U$1.7; no longer U$1.5
- net SCK: now also U$1.8; no longer U$1.7
- net SCL: now also U$1.4; no longer U$1.3
- net SDA: now also U$1.3; no longer U$1.4
Changed lines of the file:
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@@
 <?xml version="1.0" encoding="utf-8"?>
 <!DOCTYPE eagle SYSTEM "eagle.dtd">
-<eagle version="9.6.2">
+<eagle version="9.1.1">
 <drawing>
 <settings>
@@
 <net name="SCL" class="0">
 <segment>
+<pinref part="J4" gate="J1" pin="2"/>
+<wire x1="7.62" y1="-10.16" x2="12.7" y2="-10.16" width="0.1524" layer="91"/>
+<label x="7.62" y="-10.16" size="1.778" layer="95"/>
+</segment>
+<segment>
+<pinref part="J7" gate="J1" pin="2"/>
+<wire x1="38.1" y1="22.86" x2="43.18" y2="22.86" width="0.1524" layer="91"/>
+<label x="38.1" y="22.86" size="1.778" layer="95"/>
+</segment>
+<segment>
+<pinref part="U$1" gate="G$1" pin="4"/>
+<wire x1="-43.18" y1="22.86" x2="-38.1" y2="22.86" width="0.1524" layer="91"/>
+<label x="-40.64" y="22.86" size="1.778" layer="95"/>
+</segment>
+</net>
+<net name="SDA" class="0">
+<segment>
+<pinref part="J4" gate="J1" pin="1"/>
+<wire x1="7.62" y1="-12.7" x2="12.7" y2="-12.7" width="0.1524" layer="91"/>
+<label x="7.62" y="-12.7" size="1.778" layer="95"/>
+</segment>
+<segment>
+<pinref part="J7" gate="J1" pin="1"/>
+<wire x1="38.1" y1="20.32" x2="43.18" y2="20.32" width="0.1524" layer="91"/>
+<label x="38.1" y="20.32" size="1.778" layer="95"/>
+</segment>
+<segment>
 <pinref part="U$1" gate="G$1" pin="3"/>
 <wire x1="-43.18" y1="25.4" x2="-38.1" y2="25.4" width="0.1524" layer="91"/>
 <label x="-40.64" y="25.4" size="1.778" layer="95"/>
 </segment>
-<segment>
-<pinref part="J4" gate="J1" pin="2"/>
-<wire x1="7.62" y1="-10.16" x2="12.7" y2="-10.16" width="0.1524" layer="91"/>
-<label x="7.62" y="-10.16" size="1.778" layer="95"/>
-</segment>
-<segment>
-<pinref part="J7" gate="J1" pin="2"/>
-<wire x1="38.1" y1="22.86" x2="43.18" y2="22.86" width="0.1524" layer="91"/>
-<label x="38.1" y="22.86" size="1.778" layer="95"/>
-</segment>
-</net>
-<net name="SDA" class="0">
-<segment>
-<pinref part="U$1" gate="G$1" pin="4"/>
-<wire x1="-43.18" y1="22.86" x2="-38.1" y2="22.86" width="0.1524" layer="91"/>
-<label x="-40.64" y="22.86" size="1.778" layer="95"/>
-</segment>
-<segment>
-<pinref part="J4" gate="J1" pin="1"/>
-<wire x1="7.62" y1="-12.7" x2="12.7" y2="-12.7" width="0.1524" layer="91"/>
-<label x="7.62" y="-12.7" size="1.778" layer="95"/>
-</segment>
-<segment>
-<pinref part="J7" gate="J1" pin="1"/>
-<wire x1="38.1" y1="20.32" x2="43.18" y2="20.32" width="0.1524" layer="91"/>
-<label x="38.1" y="20.32" size="1.778" layer="95"/>
-</segment>
 </net>
 <net name="MISO" class="0">
+<segment>
+<pinref part="J1" gate="J1" pin="4"/>
+<wire x1="-45.72" y1="-10.16" x2="-40.64" y2="-10.16" width="0.1524" layer="91"/>
+<label x="-45.72" y="-10.16" size="1.778" layer="95"/>
+</segment>
+<segment>
+<pinref part="U$1" gate="G$1" pin="7"/>
+<wire x1="-43.18" y1="15.24" x2="-38.1" y2="15.24" width="0.1524" layer="91"/>
+<label x="-40.64" y="15.24" size="1.778" layer="95"/>
+</segment>
+</net>
+<net name="MOSI" class="0">
+<segment>
+<pinref part="U$1" gate="G$1" pin="6"/>
+<wire x1="-43.18" y1="17.78" x2="-38.1" y2="17.78" width="0.1524" layer="91"/>
+<label x="-40.64" y="17.78" size="1.778" layer="95"/>
+</segment>
+<segment>
+<pinref part="J1" gate="J1" pin="3"/>
+<wire x1="-45.72" y1="-12.7" x2="-40.64" y2="-12.7" width="0.1524" layer="91"/>
+<label x="-45.72" y="-12.7" size="1.778" layer="95"/>
+</segment>
+</net>
+<net name="SCK" class="0">
+<segment>
+<pinref part="J2" gate="J1" pin="4"/>
+<wire x1="-45.72" y1="-27.94" x2="-40.64" y2="-27.94" width="0.1524" layer="91"/>
+<label x="-45.72" y="-27.94" size="1.778" layer="95"/>
+</segment>
+<segment>
+<pinref part="U$1" gate="G$1" pin="8"/>
+<wire x1="-43.18" y1="12.7" x2="-38.1" y2="12.7" width="0.1524" layer="91"/>
+<label x="-40.64" y="12.7" size="1.778" layer="95"/>
+</segment>
+</net>
+<net name="CS" class="0">
+<segment>
+<pinref part="J1" gate="J1" pin="2"/>
+<wire x1="-45.72" y1="-15.24" x2="-40.64" y2="-15.24" width="0.1524" layer="91"/>
+<label x="-45.72" y="-15.24" size="1.778" layer="95"/>
+</segment>
 <segment>
 <pinref part="U$1" gate="G$1" pin="5"/>
@@
 <label x="-40.64" y="20.32" size="1.778" layer="95"/>
 </segment>
-<segment>
-<pinref part="J1" gate="J1" pin="4"/>
-<wire x1="-45.72" y1="-10.16" x2="-40.64" y2="-10.16" width="0.1524" layer="91"/>
-<label x="-45.72" y="-10.16" size="1.778" layer="95"/>
-</segment>
-</net>
-<net name="MOSI" class="0">
-<segment>
-<pinref part="U$1" gate="G$1" pin="6"/>
-<wire x1="-43.18" y1="17.78" x2="-38.1" y2="17.78" width="0.1524" layer="91"/>
-<label x="-40.64" y="17.78" size="1.778" layer="95"/>
-</segment>
-<segment>
-<pinref part="J1" gate="J1" pin="3"/>
-<wire x1="-45.72" y1="-12.7" x2="-40.64" y2="-12.7" width="0.1524" layer="91"/>
-<label x="-45.72" y="-12.7" size="1.778" layer="95"/>
-</segment>
-</net>
-<net name="SCK" class="0">
-<segment>
-<pinref part="U$1" gate="G$1" pin="7"/>
-<wire x1="-43.18" y1="15.24" x2="-38.1" y2="15.24" width="0.1524" layer="91"/>
-<label x="-40.64" y="15.24" size="1.778" layer="95"/>
-</segment>
-<segment>
-<pinref part="J2" gate="J1" pin="4"/>
-<wire x1="-45.72" y1="-27.94" x2="-40.64" y2="-27.94" width="0.1524" layer="91"/>
-<label x="-45.72" y="-27.94" size="1.778" layer="95"/>
-</segment>
-</net>
-<net name="CS" class="0">
-<segment>
-<pinref part="U$1" gate="G$1" pin="8"/>
-<wire x1="-43.18" y1="12.7" x2="-38.1" y2="12.7" width="0.1524" layer="91"/>
-<label x="-40.64" y="12.7" size="1.778" layer="95"/>
-</segment>
-<segment>
-<pinref part="J1" gate="J1" pin="2"/>
-<wire x1="-45.72" y1="-15.24" x2="-40.64" y2="-15.24" width="0.1524" layer="91"/>
-<label x="-45.72" y="-15.24" size="1.778" layer="95"/>
-</segment>
-</net>
+</net>

Commit message: modified:   eagle/sensors/sensors.brd
Parts:
- removed J6, J7: (no value), SparkFun-Connectors:CONN_05NO_SILK
Connections:
- removed net US_INT: J6.1
- net 3V3: no longer J7.4
- net GND: no longer J7.5
- net SCL: no longer J7.2
- net SDA: no longer J7.1
Changed lines of the file:
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@@
 <part name="J4" library="SparkFun-Connectors" deviceset="CONN_03" device="1X03_NO_SILK"/>
 <part name="J5" library="SparkFun-Connectors" deviceset="CONN_03" device="1X03_NO_SILK"/>
-<part name="J6" library="SparkFun-Connectors" deviceset="CONN_05" device="NO_SILK"/>
-<part name="J7" library="SparkFun-Connectors" deviceset="CONN_05" device="NO_SILK"/>
 </parts>
 <sheets>
@@
 <attribute name="NAME" x="-2.54" y="-19.812" size="1.778" layer="95" font="vector"/>
 </instance>
-<instance part="J6" gate="J1" x="30.48" y="5.08" smashed="yes">
-<attribute name="VALUE" x="27.94" y="-4.826" size="1.778" layer="96" font="vector"/>
-<attribute name="NAME" x="27.94" y="13.208" size="1.778" layer="95" font="vector"/>
-</instance>
-<instance part="J7" gate="J1" x="30.48" y="25.4" smashed="yes">
-<attribute name="VALUE" x="27.94" y="15.494" size="1.778" layer="96" font="vector"/>
-<attribute name="NAME" x="27.94" y="33.528" size="1.778" layer="95" font="vector"/>
-</instance>
 </instances>
 <busses>
@@
 <label x="7.62" y="-27.94" size="1.778" layer="95"/>
 </segment>
-<segment>
-<pinref part="J7" gate="J1" pin="4"/>
-<wire x1="38.1" y1="27.94" x2="43.18" y2="27.94" width="0.1524" layer="91"/>
-<label x="38.1" y="27.94" size="1.778" layer="95"/>
-</segment>
 </net>
 <net name="GND" class="0">
@@
 <label x="7.62" y="-25.4" size="1.778" layer="95"/>
 </segment>
-<segment>
-<pinref part="J7" gate="J1" pin="5"/>
-<wire x1="38.1" y1="30.48" x2="43.18" y2="30.48" width="0.1524" layer="91"/>
-<label x="38.1" y="30.48" size="1.778" layer="95"/>
-</segment>
 </net>
 <net name="SCL" class="0">
@@
 <wire x1="7.62" y1="-10.16" x2="12.7" y2="-10.16" width="0.1524" layer="91"/>
 <label x="7.62" y="-10.16" size="1.778" layer="95"/>
-</segment>
-<segment>
-<pinref part="J7" gate="J1" pin="2"/>
-<wire x1="38.1" y1="22.86" x2="43.18" y2="22.86" width="0.1524" layer="91"/>
-<label x="38.1" y="22.86" size="1.778" layer="95"/>
 </segment>
 <segment>
@@
 <wire x1="7.62" y1="-12.7" x2="12.7" y2="-12.7" width="0.1524" layer="91"/>
 <label x="7.62" y="-12.7" size="1.778" layer="95"/>
-</segment>
-<segment>
-<pinref part="J7" gate="J1" pin="1"/>
-<wire x1="38.1" y1="20.32" x2="43.18" y2="20.32" width="0.1524" layer="91"/>
-<label x="38.1" y="20.32" size="1.778" layer="95"/>
 </segment>
 <segment>
@@
 </segment>
 </net>
-<net name="US_INT" class="0">
-<segment>
-<pinref part="J6" gate="J1" pin="1"/>
-<wire x1="38.1" y1="0" x2="43.18" y2="0" width="0.1524" layer="91"/>
-<label x="38.1" y="0" size="1.778" layer="95"/>
-</segment>
-</net>
